File: Macrotype-1/Macrotype-1.kicad_pcb (KiCad board)
At the start: 2 copper layers, 115.9 x 70.6 mm, 30 parts, among them U1 ProMicro

Commit message: Update 0.3
Connections:
- MX13 pad 1: unconnected-(MX13-Pad1) -> COL1
- MX14 pad 1: unconnected-(MX14-Pad1) -> COL1
