File: Macrotype-1/Macrotype-1.kicad_sch (KiCad schematic)
At the start: 35 parts, among them SW1 SW_Push, U1 ProMicro

Commit message: Update 0.2
Parts:
- removed D15, D16, D17, D18, D19: WS2812B, LED_SMD:LED_WS2812B_PLCC4_5.0x5.0mm_P3.2mm, symbol LED:WS2812B
- removed SW1: SW_Push, symbol Switch:SW_Push
- added S1: MOMENTARY-SWITCH-SPST-SMD-6.0X3.5MM, Switches:TACTILE_SWITCH_SMD_6.0X3.5MM, symbol SparkFun-Switches:MOMENTARY-SWITCH-SPST-SMD-6.0X3.5MM
Connections:
- net COL0: now also U1.2 (D2-RX)
- net COL1: now also U1.1 (D3-TX)
- net GND: now also S1.1
- net ROW0: now also U1.6 (D0)
- net ROW1: now also U1.5 (D1)
- net ROW2: now also U1.8 (C6)
- net ROW3: now also U1.7 (D4)
- net ROW4: now also U1.10 (E6)
- net ROW5: now also U1.9 (D7)
- net ROW6: now also U1.11 (B4)
- net at U1.15 (RST): now also S1.2
- no-connect marks 1 -> 0

Commit message: Update 0.3
Parts:
- S1:  SWCH-00815 -> (none)
Connections:
- net COL1: now also MX13.1, MX14.1
Other:
- moved on the sheet: D13, D14, MX13, MX14
Changed lines of the file:
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@@
   (junction (at 129.54 93.98) (diameter 0) (color 0 0 0 0)
   )
-  (junction (at 156.21 134.62) (diameter 0) (color 0 0 0 0)
-  )
   (junction (at 142.24 96.52) (diameter 0) (color 0 0 0 0)
   )
   (junction (at 137.16 80.01) (diameter 0) (color 0 0 0 0)
   )
+  (junction (at 154.94 134.62) (diameter 0) (color 0 0 0 0)
+  )
+  (junction (at 162.56 100.33) (diameter 0) (color 0 0 0 0)
+  )
   (junction (at 162.56 60.96) (diameter 0) (color 0 0 0 0)
   )
@@
   (junction (at 129.54 74.93) (diameter 0) (color 0 0 0 0)
   )
+  (junction (at 149.86 100.33) (diameter 0) (color 0 0 0 0)
+  )
   (junction (at 149.86 80.01) (diameter 0) (color 0 0 0 0)
   )
@@
     (stroke (width 0) (type default))
   )
-  (wire (pts (xy 120.65 134.62) (xy 156.21 134.62))
+  (wire (pts (xy 120.65 134.62) (xy 154.94 134.62))
     (stroke (width 0) (type default))
   )
@@
     (stroke (width 0) (type default))
   )
+  (wire (pts (xy 154.94 134.62) (xy 167.64 134.62))
+    (stroke (width 0) (type default))
+  )
   (wire (pts (xy 162.56 55.88) (xy 162.56 60.96))
     (stroke (width 0) (type default))
   )
+  (wire (pts (xy 162.56 100.33) (xy 162.56 121.92))
+    (stroke (width 0) (type default))
+  )
   (wire (pts (xy 142.24 113.03) (xy 142.24 116.84))
     (stroke (width 0) (type default))
@@
     (stroke (width 0) (type default))
   )
+  (wire (pts (xy 149.86 100.33) (xy 149.86 121.92))
+    (stroke (width 0) (type default))
+  )
   (wire (pts (xy 142.24 77.47) (xy 167.64 77.47))
     (stroke (width 0) (type default))
@@
   )
   (wire (pts (xy 124.46 80.01) (xy 124.46 60.96))
-    (stroke (width 0) (type default))
-  )
-  (wire (pts (xy 156.21 134.62) (xy 168.91 134.62))
     (stroke (width 0) (type default))
   )
@@
     )
   )
-  (symbol (lib_id "Diode:1N4148W") (at 168.91 130.81 90) (unit 1)
-    (in_bom yes) (on_board yes) (dnp no) (fields_autoplaced)
-    (property "Reference" "D14" (at 171.45 129.54 90)
-      (effects (font (size 1.27 1.27)) (justify right))
-    )
-    (property "Value" "1N4148W" (at 171.45 132.08 90)
-      (effects (font (size 1.27 1.27)) (justify right))
-    )
-    (property "Footprint" "Diode_SMD:D_SOD-123" (at 173.355 130.81 0)
-      (effects (font (size 1.27 1.27)) hide)
-    )
-    (property "Datasheet" "https://www.vishay.com/docs/85748/1n4148w.pdf" (at 168.91 130.81 0)
-      (effects (font (size 1.27 1.27)) hide)
-    )
-    (property "Sim.Device" "D" (at 168.91 130.81 0)
-      (effects (font (size 1.27 1.27)) hide)
-    )
-    (property "Sim.Pins" "1=K 2=A" (at 168.91 130.81 0)
+  (symbol (lib_id "Diode:1N4148W") (at 167.64 130.81 90) (unit 1)
+    (in_bom yes) (on_board yes) (dnp no) (fields_autoplaced)
+    (property "Reference" "D14" (at 170.18 129.54 90)
+      (effects (font (size 1.27 1.27)) (justify right))
+    )
+    (property "Value" "1N4148W" (at 170.18 132.08 90)
+      (effects (font (size 1.27 1.27)) (justify right))
+    )
+    (property "Footprint" "Diode_SMD:D_SOD-123" (at 172.085 130.81 0)
+      (effects (font (size 1.27 1.27)) hide)
+    )
+    (property "Datasheet" "https://www.vishay.com/docs/85748/1n4148w.pdf" (at 167.64 130.81 0)
+      (effects (font (size 1.27 1.27)) hide)
+    )
+    (property "Sim.Device" "D" (at 167.64 130.81 0)
+      (effects (font (size 1.27 1.27)) hide)
+    )
+    (property "Sim.Pins" "1=K 2=A" (at 167.64 130.81 0)
       (effects (font (size 1.27 1.27)) hide)
     )
@@
       (effects (font (size 1.27 1.27)) hide)
     )
-    (property "" "SWCH-00815" (at 105.41 57.15 0)
-      (effects (font (size 1.524 1.524)))
-    )
     (pin "1")
     (pin "2")
@@
     )
   )
-  (symbol (lib_id "marbastlib-mx:MX_SW_HS") (at 153.67 124.46 0) (unit 1)
-    (in_bom yes) (on_board yes) (dnp no) (fields_autoplaced)
-    (property "Reference" "MX13" (at 153.67 116.84 0)
-      (effects (font (size 1.27 1.27)))
-    )
-    (property "Value" "MX_SW_HS" (at 153.67 119.38 0)
-      (effects (font (size 1.27 1.27)))
-    )
-    (property "Footprint" "marbastlib-mx:SW_MX_HS_1u" (at 153.67 124.46 0)
-      (effects (font (size 1.27 1.27)) hide)
-    )
-    (property "Datasheet" "~" (at 153.67 124.46 0)
+  (symbol (lib_id "marbastlib-mx:MX_SW_HS") (at 152.4 124.46 0) (unit 1)
+    (in_bom yes) (on_board yes) (dnp no) (fields_autoplaced)
+    (property "Reference" "MX13" (at 152.4 116.84 0)
+      (effects (font (size 1.27 1.27)))
+    )
+    (property "Value" "MX_SW_HS" (at 152.4 119.38 0)
+      (effects (font (size 1.27 1.27)))
+    )
+    (property "Footprint" "marbastlib-mx:SW_MX_HS_1u" (at 152.4 124.46 0)
+      (effects (font (size 1.27 1.27)) hide)
+    )
+    (property "Datasheet" "~" (at 152.4 124.46 0)
       (effects (font (size 1.27 1.27)) hide)
     )
@@
     )
   )
-  (symbol (lib_id "Diode:1N4148W") (at 156.21 130.81 90) (unit 1)
-    (in_bom yes) (on_board yes) (dnp no) (fields_autoplaced)
-    (property "Reference" "D13" (at 158.75 129.54 90)
-      (effects (font (size 1.27 1.27)) (justify right))
-    )
-    (property "Value" "1N4148W" (at 158.75 132.08 90)
-      (effects (font (size 1.27 1.27)) (justify right))
-    )
-    (property "Footprint" "Diode_SMD:D_SOD-123" (at 160.655 130.81 0)
-      (effects (font (size 1.27 1.27)) hide)
-    )
-    (property "Datasheet" "https://www.vishay.com/docs/85748/1n4148w.pdf" (at 156.21 130.81 0)
-      (effects (font (size 1.27 1.27)) hide)
-    )
-    (property "Sim.Device" "D" (at 156.21 130.81 0)
-      (effects (font (size 1.27 1.27)) hide)
-    )
-    (property "Sim.Pins" "1=K 2=A" (at 156.21 130.81 0)
+  (symbol (lib_id "Diode:1N4148W") (at 154.94 130.81 90) (unit 1)
+    (in_bom yes) (on_board yes) (dnp no) (fields_autoplaced)
+    (property "Reference" "D13" (at 157.48 129.54 90)
+      (effects (font (size 1.27 1.27)) (justify right))
+    )
+    (property "Value" "1N4148W" (at 157.48 132.08 90)
+      (effects (font (size 1.27 1.27)) (justify right))
+    )
+    (property "Footprint" "Diode_SMD:D_SOD-123" (at 159.385 130.81 0)
+      (effects (font (size 1.27 1.27)) hide)
+    )
+    (property "Datasheet" "https://www.vishay.com/docs/85748/1n4148w.pdf" (at 154.94 130.81 0)
+      (effects (font (size 1.27 1.27)) hide)
+    )
+    (property "Sim.Device" "D" (at 154.94 130.81 0)
+      (effects (font (size 1.27 1.27)) hide)
+    )
+    (property "Sim.Pins" "1=K 2=A" (at 154.94 130.81 0)
       (effects (font (size 1.27 1.27)) hide)
     )
@@
     )
   )
-  (symbol (lib_id "marbastlib-mx:MX_SW_HS") (at 166.37 124.46 0) (unit 1)
-    (in_bom yes) (on_board yes) (dnp no) (fields_autoplaced)
-    (property "Reference" "MX14" (at 166.37 116.84 0)
-      (effects (font (size 1.27 1.27)))
-    )
-    (property "Value" "MX_SW_HS" (at 166.37 119.38 0)
-      (effects (font (size 1.27 1.27)))
-    )
-    (property "Footprint" "marbastlib-mx:SW_MX_HS_1u" (at 166.37 124.46 0)
-      (effects (font (size 1.27 1.27)) hide)
-    )
-    (property "Datasheet" "~" (at 166.37 124.46 0)
-      (effects (font (size 1.27 1.27)) hide)
-    )
+  (symbol (lib_id "marbastlib-mx:MX_SW_HS") (at 165.1 124.46 0) (unit 1)
+    (in_bom yes) (on_board yes) (dnp no) (fields_autoplaced)
+    (property "Reference" "MX14" (at 165.1 116.84 0)
+      (effects (font (size 1.27 1.27)))
+    )
+    (property "Value" "MX_SW_HS" (at 165.1 119.38 0)
+      (effects (font (size 1.27 1.27)))
+    )
+    (property "Footprint" "marbastlib-mx:SW_MX_HS_1u" (at 165.1 124.46 0)
+      (effects (font (size 1.27 1.27)) hide)
+    )
+    (property "Datasheet" "~" (at 165.1 124.46 0)
+      (effects (font (size 1.27 1.27)) hide)
+    )
